File: USBhub-keyboard/USBhub-keyboard.kicad_pcb (KiCad board)
At the start: 2 copper layers, 85 parts, among them J1 Conn_01x05_Socket, J2 USB_A_v2, J3 USB_A_v2, J4 USB_C_Receptacle_USB2.0_16P_V2, J5 USB_C_Receptacle_USB2.0_16P_V2, SW1 SW_PUSH, SW10 SW_PUSH, SW11 SW_PUSH, SW12 SW_PUSH, SW13 SW_PUSH, SW14 SW_PUSH, SW15 SW_PUSH, SW16 SW_PUSH, SW2 SW_PUSH, SW3 SW_PUSH, SW4 SW_PUSH, SW5 SW_PUSH, SW6 SW_PUSH, SW7 SW_PUSH, SW8 SW_PUSH, SW9 SW_PUSH, U1 SL2.1A, U2 AZ1117-3.3, U3 RP2040, U4 W25Q16JVSS, Y1 12M/20pF/20PPM, Y2 12MHz

Commit message: a
Parts:
- added REF**: MountingHole_2.2mm_M2, MountingHole:MountingHole_2.2mm_M2, F.Cu at (163.8, 144.9)
- added REF**: MountingHole_2.2mm_M2, MountingHole:MountingHole_2.2mm_M2, F.Cu at (164.1, 37.5)
- added REF**: MountingHole_2.2mm_M2, MountingHole:MountingHole_2.2mm_M2, F.Cu at (83.4, 144.8)
- added REF**: MountingHole_2.2mm_M2, MountingHole:MountingHole_2.2mm_M2, F.Cu at (83.9, 37.7)
- BSW1, C1, C10, C11, C12, C13, C14, C15, C16, C17, C18, C19, C2, C20, C21, C22, C23, C24, C25, C26, C27, C5, C6, C7, C8, C9, D1, D10, D11, D12, D13, D14, D15, D16, D2, D3, D4, D5, D6, D7, D8, D9, FB1, R10, R11, R5, R6, R7, R8, R9, U1, U2, U3, U4, Y2: moved to B.Cu
- BSW2: value RESETSW -> RESET; moved to B.Cu
- moved C2 180.1 mm to (92.2, 62.0), turned to -90 degrees
- moved U1 168.4 mm to (112.8, 60.6), turned to -90 degrees
- moved U4 166.3 mm to (103.5, 105.7), turned to -90 degrees
- moved Y1 165.2 mm to (103.0, 56.7)
- moved C10 159.7 mm to (97.0, 52.9), turned to 90 degrees
- moved C17 156.4 mm to (116.0, 101.1), turned to 180 degrees
- moved C13 156.4 mm to (99.4, 59.1), turned to 90 degrees
- moved C8 152.1 mm to (103.8, 53.0), turned to -90 degrees
- moved U3 148.6 mm to (123.9, 105.4)
- moved R4 143.4 mm to (90.8, 48.5), turned to -90 degrees
- moved R3 139.5 mm to (93.6, 48.5), turned to -90 degrees
- moved C14 139.4 mm to (135.1, 109.9), turned to -90 degrees
- moved U2 138.8 mm to (130.2, 61.4)
- moved R1 134.8 mm to (92.3, 53.3)
- moved FB1 134.2 mm to (91.9, 52.5)
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Connections:
- C1 pad 1: +5V -> Net-(C1-Pad1)
- C2 pad 1: +5V -> Net-(C1-Pad1)
- FB1 pad 1: Net-(FB1-Pad1) -> Net-(C1-Pad1)
- J2 pad 2: DDM1 -> DDM4
- J2 pad 3: DDP1 -> DDP4
- J3 pad 2: DDM2 -> DDM3
- J3 pad 3: DDP2 -> DDP3
- J4 pad A4/B9: Net-(FB1-Pad1) -> Net-(C1-Pad1)
- J4 pad B4/A9: Net-(FB1-Pad1) -> Net-(C1-Pad1)
- J5 pad A6: DDP3 -> DDP2
- J5 pad A7: DDM3 -> DDM2
- J5 pad B6: DDP3 -> DDP2
- J5 pad B7: DDM3 -> DDM2
- R5 pad 2: DDP4 -> DDP1
- R6 pad 2: DDM4 -> DDM1
- U3 pad 15: COL2 -> unconnected-(U3-GPIO12-Pad15)
- U3 pad 16: COL3 -> unconnected-(U3-GPIO13-Pad16)
- U3 pad 29: unconnected-(U3-GPIO18-Pad29) -> COL2
- U3 pad 30: unconnected-(U3-GPIO19-Pad30) -> COL3
- U3 pad 4: ROW0 -> ROW3
- U3 pad 5: ROW1 -> ROW2
- U3 pad 53: DDM4 -> /QSPI_SD0
- U3 pad 6: ROW2 -> ROW1
- U3 pad 7: ROW3 -> ROW0
- U4 pad 5: DDM4 -> /QSPI_SD0
- Y1 pad 4: (no net) -> GND
- Y2 pad 4: (no net) -> GND
Routing:
- net /QSPI_SS: track 0.00 -> 151.4 mm, vias 0 -> 2
- net GPIO17_SCL: track 0.00 -> 149.1 mm, vias 0 -> 2
- net /RESET: track 0.00 -> 130.5 mm, vias 0 -> 2
- net GPIO16_SDA: track 0.00 -> 123.1 mm, vias 0 -> 1
- net COL0: track 0.00 -> 120.0 mm, vias 0 -> 2
- net COL3: track 0.00 -> 118.5 mm, vias 0 -> 2
- net COL2: track 0.00 -> 118.4 mm
- net ROW0: track 0.00 -> 109.1 mm, vias 0 -> 7
- net ROW3: track 0.00 -> 103.4 mm, vias 0 -> 7
- net /SWDIO: track 0.00 -> 97.8 mm, vias 0 -> 1
- net ROW1: track 0.00 -> 94.0 mm, vias 0 -> 5
- net COL1: track 0.00 -> 93.4 mm, vias 0 -> 2
- net /SWCLK: track 0.00 -> 92.7 mm, vias 0 -> 2
- net ROW2: track 0.00 -> 89.4 mm, vias 0 -> 5
- net GND: track 0.00 -> 62.1 mm, vias 0 -> 35
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- added copper zone on In2.Cu, net +3.3V
- added copper zone on In2.Cu, net +5V
- added copper zone on B.Cu, net GND
- added copper zone on F.Cu, net GND
- added copper zone on In1.Cu, net GND
Other:
- board outline added: 88.1 x 115.2 mm
- copper layers 2 -> 4

Commit message: a
Parts:
- BSW2: value RESET -> RESETSW
- C1, C11, C12, C15, C16, C18, C19, C20, C21, C22, C23, C24, C25, C5, C6, C7, C9: value 0.1µF -> 0.1uF
- C10, C13, C8: value 4.7µF -> 4.7uF
- C14, C17: value 1µF -> 1uF
- C2: value 10µF -> 10uF
- C3, C4: value 0.1µF -> 0.1uF; moved to B.Cu
- FB1: value 120Ω -> 120
- J1, R1, R2, R3, R4: moved to B.Cu
- Y1: value 12M/20pF/20PPM -> 12MHz; moved to B.Cu
- moved Y1 9.71 mm to (111.6, 52.2)
- moved C4 3.53 mm to (115.8, 52.1)
- moved R1 1.88 mm to (93.9, 54.4)
- moved C5 1.61 mm to (87.4, 45.9)
- moved C9 1.57 mm to (107.2, 52.1)
- moved R2 1.46 mm to (93.8, 57.1)
- moved FB1 0.97 mm to (91.8, 51.5)
- moved R4 0.80 mm to (90.0, 48.8)
- moved R3 0.67 mm to (93.0, 48.7)
- moved C3 0.32 mm to (131.2, 51.3)
- turned J1 to 180 degrees
Routing:
- net GPIO17_SCL: track 149.1 -> 122.0 mm, vias 2 -> 1
- net GPIO16_SDA: track 123.1 -> 117.5 mm
- net Net-(U1-VDD18): track 12.4 -> 15.6 mm
- net +5V: track 57.0 -> 59.6 mm, vias 7 -> 8
- net Net-(J4-CC1): track 5.03 -> 7.32 mm, vias 0 -> 1
- net Net-(J4-CC2): track 4.47 -> 6.19 mm, vias 0 -> 1
- net GND: track 62.1 -> 60.9 mm, vias 35 -> 34
- net Net-(J5-CC1): track 7.54 -> 8.44 mm, vias 0 -> 1
- net Net-(U1-XIN): track 5.98 -> 5.17 mm, vias 1 -> 0
- net Net-(U1-XOUT): track 9.14 -> 9.44 mm, vias 1 -> 0
- net Net-(J5-CC2): track 7.49 -> 7.38 mm, vias 0 -> 1
Other:
- board text added: "HUBboard"
- board text added: "JLCJLCJLCJLC"

Commit message: a
Routing:
- net /RESET: track 130.5 -> 111.6 mm, vias 2 -> 1
- net /SWDIO: track 98.0 -> 95.9 mm
- net GND: track 60.9 -> 59.1 mm, vias 34 -> 35
- net DDP3: track 20.4 -> 19.3 mm
- net /QSPI_SCLK: track 22.9 -> 21.9 mm
- net /QSPI_SD3: track 25.0 -> 24.0 mm
- net COL1: track 93.6 -> 94.2 mm
- net GPIO17_SCL: track 122.0 -> 121.4 mm
- net GPIO16_SDA: track 117.5 -> 116.9 mm

Commit message: a
Parts:
- removed J1: Conn_01x05_Socket, Connector_PinHeader_2.54mm:PinHeader_1x05_P2.54mm_Vertical
- added 3.3V: TestPoint, TestPoint:TestPoint_Pad_1.5x1.5mm, B.Cu at (160.4, 49.5)
- added GND: TestPoint, TestPoint:TestPoint_Pad_1.5x1.5mm, B.Cu at (160.4, 54.5)
- added RESET: TestPoint, TestPoint:TestPoint_Pad_1.5x1.5mm, B.Cu at (160.4, 59.6)
- added SWCLK: TestPoint, TestPoint:TestPoint_Pad_1.5x1.5mm, B.Cu at (160.4, 57.1)
- added SWDIO: TestPoint, TestPoint:TestPoint_Pad_1.5x1.5mm, B.Cu at (160.4, 52.0)
- BSW2: value RESETSW -> RESET
- moved C11 5.84 mm to (100.9, 59.4), turned to 180 degrees
- moved C13 5.12 mm to (100.1, 64.2), turned to 180 degrees
- moved C10 4.91 mm to (100.1, 56.8), turned to 180 degrees
- moved C9 3.60 mm to (106.2, 55.6)
- moved C12 2.06 mm to (100.9, 61.6), turned to 180 degrees
- moved C8 0.99 mm to (102.9, 52.5)
Routing:
- net GND: track 59.1 -> 49.4 mm, vias 35 -> 34
- net +5V: track 59.6 -> 53.7 mm
- net Net-(U1-VDD33): track 15.3 -> 10.9 mm
- net Net-(U1-VDD18): track 15.6 -> 12.6 mm
- net +3.3V: track 52.0 -> 53.6 mm, vias 14 -> 15
- net UDP: track 34.8 -> 36.2 mm
- net Net-(U3-USB_DM): track 60.0 -> 59.1 mm
- net UDM: track 35.3 -> 35.9 mm
- net /RESET: track 111.6 -> 111.5 mm, vias 1 -> 2
- net /SWDIO: track 95.9 -> 95.8 mm, vias 1 -> 2
