File: USBhub-keyboard/USBhub-keyboard.kicad_sch (KiCad schematic)
At the start: 22 parts, among them J2 USB_A, J3 USB_A, J4 USB_C_Receptacle_USB2.0_16P, J5 USB_C_Receptacle_USB2.0_16P, U1 SL2.1A, Y1 12M/20pF/20PPM

Commit message: a
Parts:
- removed Y1: 12M/20pF/20PPM, symbol Device:Crystal
- added C6, C7: 0.1µF, symbol Device:C
- added U2: AZ1117-3.3, symbol Regulator_Linear:AZ1117-3.3
- added Y1: 12M/20pF/20PPM, symbol Device:Crystal_GND2
- FB1: value Ferrite Bead -> 120Ω
- renumbered C12 to C10, C14 to C12, C5 to C4, C7 to C5, C10 to C8
Connections:
- net GND: now also C6.2, C7.2, U2.1 (GND), Y1.2
- net LDO5V: now reaches C12.1, C13.1, FB1.1, U1.11 (VDD5)
- net LDO5V: now also C6.1, U2.3 (VI)
- net at U1.15 (XOUT): now also Y1.1
- net at U1.16 (XIN): now also Y1.3
- new net +3V3: C7.1, U2.2 (VO)
Other:
- note added: "LDO 3.3V"

Commit message: a
Parts:
- added C14, C17: 1µF, symbol Device:C
- added C15, C16, C18, C19, C20, C21, C22, C23, C24, C25: 100nF, symbol Device:C
- added C26, C27: 18pF, symbol Device:C
- added J1: Conn_01x05_Socket, Connector_PinHeader_2.54mm:PinHeader_1x05_P2.54mm_Vertical, symbol Connector:Conn_01x05_Socket
- added R10, R11: 2.2k, symbol Device:R
- added R5, R6: 27, symbol Device:R
- added R7: DNF, symbol Device:R
- added R8: 1k, symbol Device:R
- added R9: 10k, symbol Device:R
- added SW1: BOOT, Button_Switch_SMD:SW_MEC_5GSH9, symbol Switch:SW_MEC_5E
- added SW2: SW_MEC_5E, symbol Switch:SW_MEC_5E
- added U3: RP2040, RP2040_minimal:RP2040-QFN-56, symbol MCU_RaspberryPi_RP2040:RP2040
- added U4: W25Q16JVSS, Package_SO:SOIC-8_5.3x5.3mm_P1.27mm, symbol Memory_Flash:W25Q16JVSS
- added Y2: Crystal_GND2, Crystal:Crystal_AT310_D3.0mm_L10.0mm_Horizontal_1EP_style1, symbol Device:Crystal_GND2
Connections:
- net GND: now also C14.2, C15.2, C16.2, C17.2, C18.2, C19.2, C20.2, C21.2, C22.2, C23.2, C24.2, C25.2, C26.1, C27.1, J1.3 (Pin_3), SW1.1, SW1.2, SW2.1, SW2.2, U3.19 (TESTEN), U3.57 (GND), U4.4 (GND), Y2.2
- net DDM4: now reaches U1.1 (DM4)
- net DDM4: now also R6.2, U3.53 (QSPI_SD0), U4.5 (DI/IO_{0})
- net DDP4: now reaches U1.2 (DP4)
- net DDP4: now also R5.2
- net +3V3 renamed +3.3V
- net +3.3V: now also C17.1, C18.1, C19.1, C20.1, C21.1, C22.1, C23.1, C24.1, C25.1, J1.1 (Pin_1), R10.1, R11.1, R7.1, R9.1, U3.1 (IOVDD), U3.10 (IOVDD), U3.22 (IOVDD), U3.33 (IOVDD), U3.42 (IOVDD), U3.43 (ADC_AVDD), U3.44 (VREG_IN), U3.48 (USB_VDD), U3.49 (IOVDD), U4.8 (VCC)
- new net: R6.1, U3.46 (USB_DM)
- new net: R5.1, U3.47 (USB_DP)
- new net +1V1: C14.1, C15.1, C16.1, U3.23 (DVDD), U3.45 (VREG_VOUT), U3.50 (DVDD)
- new net GPIO16_SDA: R10.2, U3.27 (GPIO16)
- new net GPIO17_SCL: R11.2, U3.28 (GPIO17)
- new net QSPI_SCLK: U3.52 (QSPI_SCLK), U4.6 (CLK)
- new net QSPI_SD1: U3.55 (QSPI_SD1), U4.2 (DO/IO_{1})
- new net QSPI_SD2: U3.54 (QSPI_SD2), U4.3 (~{WP}/IO_{2})
- new net QSPI_SD3: U3.51 (QSPI_SD3), U4.7 (~{HOLD}/~{RESET}/IO_{3})
- new net QSPI_SS: R7.2, R8.2, U3.56 (QSPI_SS), U4.1 (~{CS})
- new net RESET: J1.5 (Pin_5), R9.2, SW2.3 (K), SW2.4 (A), U3.26 (RUN)
- new net SWCLK: J1.4 (Pin_4), U3.24 (SWCLK)
- new net SWDIO: J1.2 (Pin_2), U3.25 (SWD)
- new net USB_BOOT: R8.1, SW1.3 (K), SW1.4 (A)
- new net XIN: C26.2, U3.20 (XIN), Y2.3
- new net XOUT: C27.2, U3.21 (XOUT), Y2.1
Other:
- note added: "BOOT RESET Switch"
- note added: "Crystal"
- note added: "DEBUG"
- note added: "Flash"
- note added: "I2C"
- note added: "MCU"
- moved on the sheet: C10, C11, C12, C13, C3, C4, C5, C6, C7, C8, C9, FB1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

Commit message: a
Parts:
- Y2: value Crystal_GND2 -> 12MHz
Changed lines of the file:
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@@
 			)
 		)
-		(property "Value" "Crystal_GND2"
+		(property "Value" "12MHz"
 			(at 226.06 163.8299 90)
 			(show_name no)

Commit message: a
Parts:
- removed J2, J3: USB_A, symbol Connector:USB_A
- removed J4, J5: USB_C_Receptacle_USB2.0_16P, symbol Connector:USB_C_Receptacle_USB2.0_16P
- added D1, D10, D11, D12, D13, D14, D15, D16, D2, D3, D4, D5, D6, D7, D8, D9: 1N4148W, Diode_SMD:D_SOD-123, symbol Diode:1N4148W
- added J2, J3: USB_A_v2, USB-A:3210W1BCE, symbol USB-A:USB_A_v2
- added J4, J5: USB_C_Receptacle_USB2.0_16P_V2, USB-C:CONN_8p94X6p5X3p16_12L_GCC, symbol USB-C:USB_C_Receptacle_USB2.0_16P_V2
- added OL1: OLED, SSD1306:128x64OLED, symbol BrownSugar_KBD:OLED
- added SW1, SW10, SW11, SW12, SW13, SW14, SW15, SW16, SW2, SW3, SW4, SW5, SW6, SW7, SW8, SW9: SW_PUSH, BrownSugar_KBD:CherryMX_Hotswap_via_1U, symbol BrownSugar_KBD:SW_PUSH
- BSW1: renamed from SW1; footprint Button_Switch_SMD:SW_MEC_5GSH9 -> TS04-66-50-BK-260-SMT:SW_TS04-66-50-BK-260-SMT
- BSW2: renamed from SW2; value SW_MEC_5E -> RESETSW; footprint (none) -> TS04-66-50-BK-260-SMT:SW_TS04-66-50-BK-260-SMT
- C1, C11, C12, C26, C27, C3, C4, C5, C6, C7, C9: footprint (none) -> Capacitor_SMD:C_0603_1608Metric
- C10, C13, C8: footprint (none) -> Capacitor_SMD:C_1206_3216Metric
- C14, C17, C2: footprint (none) -> Capacitor_SMD:C_0805_2012Metric
- C15, C16, C18, C19, C20, C21, C22, C23, C24, C25: value 100nF -> 0.1µF; footprint (none) -> Capacitor_SMD:C_0603_1608Metric
- FB1, R1, R10, R11, R2, R3, R4, R5, R6, R7, R8, R9: footprint (none) -> Resistor_SMD:R_0603_1608Metric
- U2: footprint (none) -> Package_TO_SOT_SMD:SOT-223-3_TabPin2
- U3: footprint RP2040_minimal:RP2040-QFN-56 -> RP2040_minimal_r2:RP2040-QFN-56
- Y1: footprint (none) -> Crystal:Crystal_SMD_3225-4Pin_3.2x2.5mm
- Y2: footprint Crystal:Crystal_AT310_D3.0mm_L10.0mm_Horizontal_1EP_style1 -> Crystal:Crystal_SMD_3225-4Pin_3.2x2.5mm
Connections:
- net +3.3V: now also OL1.3 (VCC)
- net +5V: now also C12.1, C13.1, C6.1, U1.11 (VDD5), U2.3 (VI), J2.1 (VBUS), J3.1 (VBUS), J5.A4/B9 (VBUS), J5.A9 (VBUS), J5.B4 (VBUS), J5.B4/A9 (VBUS), J5.B9 (VBUS)
- net DDM1: now also J2.2 (D-)
- net DDM2: now also J3.2 (D-)
- net DDM3: now also J5.A7 (D-), J5.B7 (D-)
- net DDP1: now also J2.3 (D+)
- net DDP2: now also J3.3 (D+)
- net DDP3: now also J5.A6 (D+), J5.B6 (D+)
- net GND: now also J2.4 (GND), J2.5 (Shield), J2.6 (Shield), J3.4 (GND), J3.5 (Shield), J3.6 (Shield), J4.13 (SHIELD), J4.14 (SHIELD), J4.15 (SHIELD), J4.16 (SHIELD), J4.A1/B12 (GND), J4.A12 (GND), J4.B1 (GND), J4.B1/A12 (GND), J4.B12 (GND), J5.13 (SHIELD), J5.14 (SHIELD), J5.15 (SHIELD), J5.16 (SHIELD), J5.A1/B12 (GND), J5.A12 (GND), J5.B1 (GND), J5.B1/A12 (GND), J5.B12 (GND), OL1.4 (GND)
- net GPIO16_SDA: now also OL1.1 (SDA)
- net GPIO17_SCL: now also OL1.2 (SCL)
- net UDM: now also J4.A7 (D-), J4.B7 (D-)
- net UDP: now also J4.A6 (D+), J4.B6 (D+)
- net COL0: now reaches U3.13 (GPIO10)
- net COL0: now also SW1.1, SW13.1, SW5.1, SW9.1
- net COL1: now reaches U3.14 (GPIO11)
- net COL1: now also SW10.1, SW14.1, SW2.1, SW6.1
- net COL2: now reaches U3.15 (GPIO12)
- net COL2: now also SW11.1, SW15.1, SW3.1, SW7.1
- net COL3: now reaches U3.16 (GPIO13)
- net COL3: now also SW12.1, SW16.1, SW4.1, SW8.1
- net ROW0: now reaches U3.4 (GPIO2)
- net ROW0: now also D1.1 (K), D2.1 (K), D3.1 (K), D4.1 (K)
- net ROW1: now reaches U3.5 (GPIO3)
- net ROW1: now also D5.1 (K), D6.1 (K), D7.1 (K), D8.1 (K)
- net ROW2: now reaches U3.6 (GPIO4)
- net ROW2: now also D10.1 (K), D11.1 (K), D12.1 (K), D9.1 (K)
- net ROW3: now reaches U3.7 (GPIO5)
- net ROW3: now also D13.1 (K), D14.1 (K), D15.1 (K), D16.1 (K)
- net at R1.1: now also J4.A5 (CC1)
- net at R2.1: now also J4.B5 (CC2)
- net at R4.1: now also J5.B5 (CC2)
- net at R3.1: now also J5.A5 (CC1)
- removed net LDO5V: C12.1, C13.1, C6.1, FB1.1, U1.11 (VDD5), U2.3 (VI)
- new net: D15.2 (A), SW15.2
- new net: D16.2 (A), SW16.2
- new net: D6.2 (A), SW6.2
- new net: FB1.1, J4.A4/B9 (VBUS), J4.A9 (VBUS), J4.B4 (VBUS), J4.B4/A9 (VBUS), J4.B9 (VBUS)
- new net: D7.2 (A), SW7.2
- new net: D8.2 (A), SW8.2
- new net: D2.2 (A), SW2.2
- new net: D11.2 (A), SW11.2
- new net: D4.2 (A), SW4.2
- new net: D5.2 (A), SW5.2
- new net: D1.2 (A), SW1.2
- new net: D13.2 (A), SW13.2
- new net: D10.2 (A), SW10.2
- new net: D3.2 (A), SW3.2
- new net: D9.2 (A), SW9.2
- new net: D14.2 (A), SW14.2
- new net: D12.2 (A), SW12.2
- no-connect marks 4 -> 24
Other:
- note added: "Keyboard SW"
- note added: "OLED"
- moved on the sheet: FB1

Commit message: a
Connections:
- net +5V: no longer C1.1, C2.1
- net COL2: now also U3.29 (GPIO18); no longer U3.15 (GPIO12)
- net COL3: now also U3.30 (GPIO19); no longer U3.16 (GPIO13)
- net DDM1: now also R6.2; no longer J2.2 (D-)
- net DDM2: now also J5.A7 (D-), J5.B7 (D-); no longer J3.2 (D-)
- net DDM3: now also J3.2 (D-); no longer J5.A7 (D-), J5.B7 (D-)
- net DDM4: now also J2.2 (D-); no longer R6.2, U3.53 (QSPI_SD0), U4.5 (DI/IO_{0})
- net DDP1: now also R5.2; no longer J2.3 (D+)
- net DDP2: now also J5.A6 (D+), J5.B6 (D+); no longer J3.3 (D+)
- net DDP3: now also J3.3 (D+); no longer J5.A6 (D+), J5.B6 (D+)
- net DDP4: now also J2.3 (D+); no longer R5.2
- net ROW0: now also U3.7 (GPIO5); no longer U3.4 (GPIO2)
- net ROW1: now also U3.6 (GPIO4); no longer U3.5 (GPIO3)
- net ROW2: now also U3.5 (GPIO3); no longer U3.6 (GPIO4)
- net ROW3: now also U3.4 (GPIO2); no longer U3.7 (GPIO5)
- net at FB1.1, J4.A4/B9 (VBUS), J4.A9 (VBUS)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: now also C1.1, C2.1
- new net QSPI_SD0: U3.53 (QSPI_SD0), U4.5 (DI/IO_{0})
Other:
- moved on the sheet: FB1

Commit message: a
Parts:
- C1, C11, C12, C15, C16, C18, C19, C20, C21, C22, C23, C24, C25, C3, C4, C5, C6, C7, C9: value 0.1µF -> 0.1uF
- C10, C13, C8: value 4.7µF -> 4.7uF
- C14, C17: value 1µF -> 1uF
- C2: value 10µF -> 10uF
- FB1: value 120Ω -> 120
- Y1: value 12M/20pF/20PPM -> 12MHz
Changed lines of the file:
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@@
 			)
 		)
-		(property "Value" "120Ω"
+		(property "Value" "120"
 			(at 84.582 29.21 90)
 			(show_name no)
@@
 			)
 		)
-		(property "Value" "0.1µF"
+		(property "Value" "0.1uF"
 			(at 255.27 53.3399 0)
 			(show_name no)
@@
 			)
 		)
-		(property "Value" "0.1µF"
+		(property "Value" "0.1uF"
 			(at 80.264 40.64 0)
 			(show_name no)
@@
 			)
 		)
-		(property "Value" "0.1µF"
+		(property "Value" "0.1uF"
 			(at 156.21 78.7399 0)
 			(show_name no)
@@
 			)
 		)
-		(property "Value" "0.1µF"
+		(property "Value" "0.1uF"
 			(at 394.97 40.6399 0)
 			(show_name no)
@@
 			)
 		)
-		(property "Value" "0.1µF"
+		(property "Value" "0.1uF"
 			(at 326.39 40.6399 0)
 			(show_name no)
@@
 			)
 		)
-		(property "Value" "0.1µF"
+		(property "Value" "0.1uF"
 			(at 366.014 234.95 0)
 			(show_name no)
@@
 			)
 		)
-		(property "Value" "4.7µF"
+		(property "Value" "4.7uF"
 			(at 91.44 126.746 0)
 			(show_name no)
@@
 			)
 		)
-		(property "Value" "0.1µF"
+		(property "Value" "0.1uF"
 			(at 372.11 40.6399 0)
 			(show_name no)
@@
 			)
 		)
-		(property "Value" "0.1µF"
+		(property "Value" "0.1uF"
 			(at 308.61 40.6399 0)
 			(show_name no)
@@
 			)
 		)
-		(property "Value" "1µF"
+		(property "Value" "1uF"
 			(at 356.87 52.0699 0)
 			(show_name no)
@@
 			)
 		)
-		(property "Value" "0.1µF"
+		(property "Value" "0.1uF"
 			(at 349.25 40.6399 0)
 			(show_name no)
@@
 			)
 		)
-		(property "Value" "0.1µF"
+		(property "Value" "0.1uF"
 			(at 297.18 40.6399 0)
 			(show_name no)
@@
 			)
 		)
-		(property "Value" "0.1µF"
+		(property "Value" "0.1uF"
 			(at 165.354 115.316 0)
 			(show_name no)
@@
 			)
 		)
-		(property "Value" "0.1µF"
+		(property "Value" "0.1uF"
 			(at 156.21 43.1799 0)
 			(show_name no)
@@
 			)
 		)
-		(property "Value" "4.7µF"
+		(property "Value" "4.7uF"
 			(at 91.44 114.3 0)
 			(show_name no)
@@
 			)
 		)
-		(property "Value" "0.1µF"
+		(property "Value" "0.1uF"
 			(at 383.54 40.6399 0)
 			(show_name no)
@@
 			)
 		)
-		(property "Value" "0.1µF"
+		(property "Value" "0.1uF"
 			(at 337.82 40.6399 0)
 			(show_name no)
@@
 			)
 		)
-		(property "Value" "12M/20pF/20PPM"
+		(property "Value" "12MHz"
 			(at 83.82 101.092 90)
 			(show_name no)
@@
 			)
 		)
-		(property "Value" "0.1µF"
+		(property "Value" "0.1uF"
 			(at 339.852 234.696 0)
 			(show_name no)
@@
 			)
 		)
-		(property "Value" "10µF"
+		(property "Value" "10uF"
 			(at 90.678 40.64 0)
 			(show_name no)
@@
 			)
 		)
-		(property "Value" "1µF"
+		(property "Value" "1uF"
 			(at 304.8 52.0699 0)
 			(show_name no)
@@
 			)
 		)
-		(property "Value" "0.1µF"
+		(property "Value" "0.1uF"
 			(at 82.042 126.492 0)
 			(show_name no)
@@
 			)
 		)
-		(property "Value" "4.7µF"
+		(property "Value" "4.7uF"
 			(at 80.264 149.86 0)
 			(show_name no)
@@
 			)
 		)
-		(property "Value" "0.1µF"
+		(property "Value" "0.1uF"
 			(at 360.68 40.6399 0)
 			(show_name no)
@@
 			)
 		)
-		(property "Value" "0.1µF"
+		(property "Value" "0.1uF"
 			(at 88.9 149.86 0)
 			(show_name no)
@@
 			)
 		)
-		(property "Value" "0.1µF"
+		(property "Value" "0.1uF"
 			(at 82.296 114.046 0)
 			(show_name no)

Commit message: a
Parts:
- removed J1: Conn_01x05_Socket, Connector_PinHeader_2.54mm:PinHeader_1x05_P2.54mm_Vertical, symbol Connector:Conn_01x05_Socket
- added TP1, TP2, TP3, TP4, TP5: TestPoint, TestPoint:TestPoint_Pad_1.5x1.5mm, symbol Connector:TestPoint
- BSW2: value RESETSW -> RESET
Connections:
- net +3.3V: now also TP1.1
- net GND: now also TP3.1
- net RESET: now also TP5.1
- net SWCLK: now also TP4.1
- net SWDIO: now also TP2.1
